Commit message: Visaul feedback for the ball is implemented.

File: gopigo_description/urdf/ball.urdf.xacro (robot description, xacro)
@@ -4,5 +4,5 @@
   <link name="ball_base"></link>
   <joint name="ball_joint" type="fixed">
-    <origin xyz="0.5 0 0" rpy="0 0 0" />
+    <origin xyz="0 0 0" rpy="0 0 0" />
     <parent link="ball_base"/>
     <child link="ball_base_link" />

File: gopigo_description/urdf/base/0_0_0/gopigo_base.urdf.xacro (robot description, xacro)
@@ -77,5 +77,5 @@
       </inertial>
     </link>
-    <xacro:marker_0 name="marker0" pad_base="base" marker_pos="0 0 ${H/2}" marker_ori="0 0 0" scale="1.0"/>
+    <xacro:marker_0 name="marker0" pad_base="base" marker_pos="0 0 ${H/2}" marker_ori="0 0 0" scale="1.5"/>
   </xacro:macro>
 </robot>

File: gopigo_description/urdf/football_field.urdf.xacro (robot description, xacro)
@@ -2,6 +2,6 @@
 <robot name="field" xmlns:xacro="http://www.ros.org/wiki/xacro">
   <material name="green"><color rgba="0.0 1.0 0.0 1.0" /></material>
-  <xacro:property name="w"         value= "2.0"/> <!-- [m] -->
-  <xacro:property name="l"         value= "1.5"/> <!-- [m] -->
+  <xacro:property name="w"         value= "2.5"/> <!-- [m] -->
+  <xacro:property name="l"         value= "2.0"/> <!-- [m] -->
   <xacro:property name="wall_w"    value= "0.02"/> <!-- [m] -->
   <link name="field_base"></link>
@@ -16,5 +16,5 @@
       <origin xyz="0 0 0" rpy="0 0 0" />
       <geometry>
-        <box size="${w} ${l} 0.0005"/>
+        <box size="${w} ${l} 0.003"/>
       </geometry>
       <material name="green" />
@@ -23,5 +23,5 @@
       <origin xyz="0 0 0"/>
       <geometry>
-        <box size="${w} ${l} 0.0005"/>
+        <box size="${w} ${l} 0.003"/>
       </geometry>
     </collision>

File: gopigo_description/urdf/overhead_camera.urdf.xacro (robot description, xacro)
@@ -7,5 +7,5 @@
   <xacro:property name="pole_thickness"         value= "0.05"/> <!-- [m] -->
   <xacro:property name="pole_height"         value= "1.0"/> <!-- [m] -->
-  <xacro:property name="vpole_height"         value= "1.0"/> <!-- [m] -->
+  <xacro:property name="vpole_height"         value= "1.5"/> <!-- [m] -->
   <xacro:property name="camera_w"         value= "0.1"/> <!-- [m] -->
   <xacro:property name="camera_l"         value= "0.1"/> <!-- [m] -->
@@ -92,5 +92,5 @@
   </link>
   <!-- Camera link -->
-  <joint name="camera_top_joint" type="revolute">
+  <joint name="camera_top_joint" type="fixed">
     <origin xyz="0 0 ${-vpole_height/2}" rpy="0 0 -1.57" />
     <parent link="v_pole"/>
