Commit message: new tutorial files are added

File: gopigo_description/urdf/base/0_0_0/gopigo_base.urdf.xacro (robot description, xacro)
@@ -77,5 +77,5 @@
       </inertial>
     </link>
-    <xacro:marker_0 name="marker0" pad_base="base" marker_pos="0 0 ${H/2}" marker_ori="0 0 0" scale="1"/>
+    <xacro:marker_0 name="marker0" pad_base="base" marker_pos="0 0 ${H/2}" marker_ori="0 0 0" scale="1.5"/>
   </xacro:macro>
 </robot>

File: gopigo_description/urdf/overhead_camera.urdf.xacro (robot description, xacro)
@@ -4,11 +4,14 @@
   <material name="white"><color rgba="1.0 1.0 1.0 1.0" /></material>
   <!-- Camera plugin -->
-  <xacro:include filename="$(find cri_efe_description)/urdf/include/camera.gazebo.xacro" />
+  <xacro:include filename="$(find gopigo_description)/urdf/include/camera.gazebo.xacro" />
   <xacro:property name="pole_thickness"         value= "0.05"/> <!-- [m] -->
-  <xacro:property name="pole_height"         value= "1.5"/> <!-- [m] -->
-  <xacro:property name="vpole_height"         value= "1.5"/> <!-- [m] -->
+  <xacro:property name="pole_height"         value= "1.0"/> <!-- [m] -->
+  <xacro:property name="vpole_height"         value= "1.0"/> <!-- [m] -->
   <xacro:property name="camera_w"         value= "0.1"/> <!-- [m] -->
   <xacro:property name="camera_l"         value= "0.1"/> <!-- [m] -->
   <xacro:property name="camera_h"         value= "0.5"/> <!-- [m] -->
+  <xacro:property name="lens_x"     value= "0.0"/> <!-- [m] -->
+  <xacro:property name="lens_y"     value= "0.0"/> <!-- [m] -->
+  <xacro:property name="lens_z"     value= "0.0"/> <!-- [m] -->
   <link name="camera_base"></link>
   <!-- Camera link -->
@@ -116,4 +119,14 @@
     </inertial>
   </link>
+  <joint name="camera_optical_joint" type="fixed">
+    <!-- these values have to be these values otherwise the gazebo camera
+        image won't be aligned properly with the frame it is supposedly
+        originating from -->
+    <origin xyz="${lens_x} ${lens_y} ${lens_z}" rpy="${-pi/2} 0 ${-pi/2}"/>
+    <parent link="camera_link"/>
+    <child link="camera_link_optical"/>
+  </joint>
+  <link name="camera_link_optical">
+  </link>
   <gazebo reference="camera_link" >
       <material>Gazebo/Black</material>

Commit message: simulation for only gopigo is prepared and new football simulation is created

File: gopigo_description/urdf/base/0_0_0/gopigo_base.urdf.xacro (robot description, xacro)
@@ -77,5 +77,5 @@
       </inertial>
     </link>
-    <xacro:marker_0 name="marker0" pad_base="base" marker_pos="0 0 ${H/2}" marker_ori="0 0 0" scale="1.5"/>
+    <xacro:marker_0 name="marker0" pad_base="base" marker_pos="0 0 ${H/2}" marker_ori="0 0 0" scale="1.0"/>
   </xacro:macro>
 </robot>

File: gopigo_description/urdf/base/0_0_0/gopigo_base_parameters.urdf.xacro (robot description, xacro)
@@ -10,4 +10,4 @@
   <xacro:property name="L"   value= "0.2"/> <!-- [m] -->
   <xacro:property name="W"   value= "0.1"/> <!-- [m] -->
-  <xacro:property name="H"   value= "0.1"/> <!-- [m] -->
+  <xacro:property name="H"   value= "0.08"/> <!-- [m] -->
 </robot>

Commit message: multi_robot simulation

File: gopigo_description/urdf/base/0_0_0/gopigo_base.urdf.xacro (robot description, xacro)
@@ -2,6 +2,13 @@
 <robot xmlns:xacro="http://www.ros.org/wiki/xacro">
   <xacro:include filename="$(find gopigo_description)/urdf/single_markers/marker_0.urdf.xacro"/>
+  <xacro:include filename="$(find gopigo_description)/urdf/single_markers/marker_1.urdf.xacro"/>
+  <xacro:include filename="$(find gopigo_description)/urdf/single_markers/marker_2.urdf.xacro"/>
+  <xacro:include filename="$(find gopigo_description)/urdf/single_markers/marker_3.urdf.xacro"/>
+  <xacro:include filename="$(find gopigo_description)/urdf/single_markers/marker_4.urdf.xacro"/>
+  <xacro:include filename="$(find gopigo_description)/urdf/single_markers/marker_5.urdf.xacro"/>
+  <xacro:include filename="$(find gopigo_description)/urdf/single_markers/marker_6.urdf.xacro"/>
+  <xacro:include filename="$(find gopigo_description)/urdf/single_markers/marker_7.urdf.xacro"/>
   <!-- Base -->
-  <xacro:macro name="gopigo_base"  params="name **properties">
+  <xacro:macro name="gopigo_base"  params="name robot_name **properties">
     <!-- Xacro:Properties-->
     <xacro:insert_block name="properties"/>
@@ -9,6 +16,6 @@
     <xacro:if value="$(arg fixed)">
       <gazebo>
-        <joint name="world_joint" type="fixed">
-          <parent>${name}</parent>
+        <joint name="${robot_name}_world_joint" type="fixed">
+          <parent>${robot_name}_${name}</parent>
           <child>world</child>
         </joint>
@@ -16,5 +23,5 @@
     </xacro:if>
     <!-- Base link -->
-    <link name="${name}">
+    <link name="${robot_name}_${name}">
       <visual>
         <origin xyz="0 0 0" rpy="0 0 0"/>
@@ -31,10 +38,10 @@
       </collision>
     </link>
-    <joint name="${name}_to_dummy_wheel_front" type="fixed">
-      <parent link="${name}"/>
-      <child link="dummy_wheel_front"/>
+    <joint name="${robot_name}_${name}_to_dummy_wheel_front" type="fixed">
+      <parent link="${robot_name}_${name}"/>
+      <child link="${robot_name}_dummy_wheel_front"/>
       <origin xyz="0.10 0 -0.05" rpy="0 0 0"/>
     </joint>
-    <link name="dummy_wheel_front">
+    <link name="${robot_name}_dummy_wheel_front">
       <visual>
         <origin xyz="0 0 0" rpy="0 0 0"/>
@@ -51,5 +58,5 @@
       </collision>
     </link>
-    <gazebo reference="dummy_wheel_front" >
+    <gazebo reference="${robot_name}_dummy_wheel_front" >
     	<kp>1000000.0</kp>
         <kd>100.0</kd>
@@ -62,11 +69,11 @@
     </gazebo>
     <!-- Fixed joint to add dummy inertia link -->
-    <joint name="${name}_to_${name}_inertia" type="fixed">
-      <parent link="${name}"/>
-      <child link="${name}_inertia"/>
+    <joint name="${robot_name}_${name}_to_${name}_inertia" type="fixed">
+      <parent link="${robot_name}_${name}"/>
+      <child link="${robot_name}_${name}_inertia"/>
       <origin xyz="0 0 0" rpy="0 0 0"/>
     </joint>
     <!-- Dummy inertia link, because KDL cannot have inertia on the base link -->
-    <link name="${name}_inertia">
+    <link name="${robot_name}_${name}_inertia">
       <inertial>
         <origin   xyz="0 0 0"
@@ -77,5 +84,28 @@
       </inertial>
     </link>
-    <xacro:marker_0 name="marker0" pad_base="base" marker_pos="0 0 ${H/2}" marker_ori="0 0 0" scale="1.5"/>
+    <xacro:if value="${robot_name.endswith('0000')}">
+      <xacro:marker_0 name="marker0" pad_base="${robot_name}_base" marker_pos="0 0 ${H/2}" marker_ori="0 0 0" scale="1.5"/>
+    </xacro:if>
+    <xacro:if value="${robot_name.endswith('0001')}">
+      <xacro:marker_1 name="marker1" pad_base="${robot_name}_base" marker_pos="0 0 ${H/2}" marker_ori="0 0 0" scale="1.5"/>
+    </xacro:if>
+    <xacro:if value="${robot_name.endswith('0002')}">
+      <xacro:marker_2 name="marker2" pad_base="${robot_name}_base" marker_pos="0 0 ${H/2}" marker_ori="0 0 0" scale="1.5"/>
+    </xacro:if>
+    <xacro:if value="${robot_name.endswith('0003')}">
+      <xacro:marker_3 name="marker3" pad_base="${robot_name}_base" marker_pos="0 0 ${H/2}" marker_ori="0 0 0" scale="1.5"/>
+    </xacro:if>
+    <xacro:if value="${robot_name.endswith('0004')}">
+      <xacro:marker_4 name="marker4" pad_base="${robot_name}_base" marker_pos="0 0 ${H/2}" marker_ori="0 0 0" scale="1.5"/>
+    </xacro:if>
+    <xacro:if value="${robot_name.endswith('0005')}">
+      <xacro:marker_5 name="marker5" pad_base="${robot_name}_base" marker_pos="0 0 ${H/2}" marker_ori="0 0 0" scale="1.5"/>
+    </xacro:if>
+    <xacro:if value="${robot_name.endswith('0006')}">
+      <xacro:marker_6 name="marker6" pad_base="${robot_name}_base" marker_pos="0 0 ${H/2}" marker_ori="0 0 0" scale="1.5"/>
+    </xacro:if>
+    <xacro:if value="${robot_name.endswith('0007')}">
+      <xacro:marker_7 name="marker7" pad_base="${robot_name}_base" marker_pos="0 0 ${H/2}" marker_ori="0 0 0" scale="1.5"/>
+    </xacro:if>
   </xacro:macro>
 </robot>

File: gopigo_description/urdf/gopigo.urdf.xacro (robot description, xacro)
@@ -3,5 +3,5 @@
 <robot name="gopigo" xmlns:xacro="http://www.ros.org/wiki/xacro">
   <!-- Arguments -->
-  <xacro:arg name="robot_name"          default="gopigo0000"/>
+  <xacro:arg name="robot_name"          default="gopigo_0000"/>
   <xacro:arg name="simulation"          default="true"/>
   <xacro:arg name="fixed"               default="false"/>
@@ -10,4 +10,5 @@
   <!-- Component versions -->
   <xacro:property name="base_version"    value="0_0_0"/>
+  <xacro:property name="robot_name" value="$(arg robot_name)" />
   <!-- Includes -->
   <xacro:include filename="$(find gopigo_description)/urdf/include/gopigo_utils.urdf.xacro"/>
@@ -15,5 +16,5 @@
   <xacro:include filename="$(find gopigo_description)/urdf/wheel/wheel.urdf.xacro"/>
   <!-- Base -->
-  <xacro:gopigo_base name="base">
+  <xacro:gopigo_base robot_name="${robot_name}" name="base">
     <properties>
       <xacro:include filename="$(find gopigo_description)/urdf/base/${base_version}/gopigo_base_parameters.urdf.xacro"/>
@@ -21,5 +22,5 @@
   </xacro:gopigo_base>
   <!-- Left components -->
-  <xacro:wheel side="L">
+  <xacro:wheel robot_name="${robot_name}" side="L">
     <properties>
       <xacro:include filename="$(find gopigo_description)/urdf/wheel/wheel_parameters.urdf.xacro"/>
@@ -27,5 +28,5 @@
   </xacro:wheel>
   <!-- Right components -->
-  <xacro:wheel side="R">
+  <xacro:wheel robot_name="${robot_name}" side="R">
     <properties>
       <xacro:include filename="$(find gopigo_description)/urdf/wheel/wheel_parameters.urdf.xacro"/>

File: gopigo_description/urdf/wheel/wheel.urdf.xacro (robot description, xacro)
@@ -2,5 +2,5 @@
 <robot xmlns:xacro="http://www.ros.org/wiki/xacro">
   <!-- Wheel -->
-  <xacro:macro name="wheel"  params="side **properties">
+  <xacro:macro name="wheel"  params="side robot_name **properties">
     <!-- Xacro:Properties-->
     <xacro:insert_block name="properties"/>
@@ -8,5 +8,5 @@
     <xacro:property name="front" value="${int(side.startswith('F', 1))*2-1}"/>
     <!-- Wheel link -->
-    <link name="${side}_WHEEL">
+    <link name="${robot_name}_${side}_WHEEL">
       <visual>
         <origin xyz="0 0 0" rpy="0 0 0"/>
@@ -30,11 +30,11 @@
       </inertial>
     </link>
-    <joint name="${side}_WH" type="continuous">
-      <parent link="base"/>
-      <child link="${side}_WHEEL"/>
+    <joint name="${robot_name}_${side}_WH" type="continuous">
+      <parent link="${robot_name}_base"/>
+      <child link="${robot_name}_${side}_WHEEL"/>
       <origin xyz="${front * x_wheel} ${left * y_wheel} ${z_wheel}" rpy="${PI/2} 0 0"/>
       <axis xyz="0 0 1" />
     </joint>
-    <gazebo reference="${side}_WH" >
+    <gazebo reference="${robot_name}_${side}_WH" >
     	<kp>${kp_wheel}</kp>
         <kd>${kd_wheel}</kd>
